File: Engineering/2022-2023 Rocket/Avionics/Io_Design/_autosave-Io.kicad_pcb (KiCad board)
At the start: 2 copper layers, 71 parts, among them IC1 AP63300WU-7, IC2 BMP390, J1 PH1-04-UA, J2 TB002-500-08BE, J3 PH1-04-UA, J4 TB002-500-02BE, J5 TB002-500-02BE, J6 MEM2075-00-140-01-A, J7 KMMX-BSMT35S-B30TR, J8 0732511151, Q1 DMG2301L, Q2 CSD17578Q5A, Q3 CSD17578Q5A, Q4 CSD17578Q5A, Q5 CSD17578Q5A, SW1 LSSM12-40-P-V-T/R, U1 LD39150DT33, U2 STM32L486RGT7, U3 USBLC6-2SC6, U4 LSM6DSO32TR, U5 RFM95W-915S2, U6 SAM-M8Q-0-10, Y1 ECS-400-10-37B2-CKM-TR

Commit message: Intermediate avionics update
Parts:
- moved C3 23.6 mm to (106.7, 55.9)
- moved C5 23.6 mm to (101.6, 53.3)
- moved IC1 23.6 mm to (103.7, 55.9)
- moved R14 23.6 mm to (111.8, 76.6)
- moved R15 23.6 mm to (111.8, 73.7)
- moved C1 23.6 mm to (99.1, 56.7)
- moved C7 23.6 mm to (109.2, 73.7)
- moved L1 23.6 mm to (105.4, 64.8)
- moved C6 23.6 mm to (106.9, 73.7)
- moved C20 16.6 mm to (105.4, 77.5)
- moved C17 12.2 mm to (102.9, 95.2), turned to 180 degrees
- moved C16 11.9 mm to (102.9, 92.7), turned to 180 degrees
- moved U4 9.30 mm to (102.9, 80.0), turned to 180 degrees
- moved C21 8.91 mm to (101.9, 77.0)
- moved U3 6.63 mm to (118.1, 73.7)
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Routing:
- net ARM: track 4.53 -> 3.73 mm
