File: Engineering/2022-2023 Rocket/Avionics/Io_Design/Io.kicad_sch (KiCad schematic)
At the start: 32 parts, among them IC1 AP63300WU-7, SW1 SW_SPDT, U1 STM32L486RGT7, Y1 ECS-400-10-37B2-CKM-TR

Commit message: Finished schematic
Parts:
- removed R? (x2): 47K, symbol Device:R
- removed R?: 10K, symbol Device:R
- added C12, C20, C21, C22, C23, C24, C25, C26: 100nf, Capacitor_SMD:C_0402_1005Metric, symbol Device:C
- added C17: 10n, Capacitor_SMD:C_0402_1005Metric, symbol Device:C
- added C18, C19: 1u, Capacitor_SMD:C_0402_1005Metric, symbol Device:C
- added D2: LTST-C190KRKT, symbol Device:LED
- added FB1: 120R, symbol Device:FerriteBead
- added IC2: BMP390, BMP390, symbol Io_Symbols:BMP390
- added J1, J4: PH1-04-UA, symbol Connector:Conn_01x04_Male
- added J2: MEM2075-00-140-01-A, symbol Connector:Micro_SD_Card_Det
- added J3: TB002-500-08BE, symbol Connector:Screw_Terminal_01x08
- added J5, J6: TB002-500-02BE, symbol Connector:Screw_Terminal_01x02
- added J8: EMPCB.SMAFSTJ.B.HT, symbol Connector:Conn_Coaxial
- added Q2, Q3, Q4, Q5: CSD17578Q5A, Package_TO_SOT_SMD:TDSON-8-1, symbol Transistor_FET:CSD17578Q5A
- added R10, R12, R14, R16: 30.1k, symbol Device:R
- added R11, R13, R15, R17: 60k, symbol Device:R
- added R2, R3, R4, R5: 1K, symbol Device:R
- added R20, R22: 1.5k, symbol Device:R
- added R6, R7, R8, R9: 100K, symbol Device:R
- added U3: SAM-M8Q-0-10, RF_GPS:ublox_SAM-M8Q, symbol RF_GPS:SAM-M8Q
- added U4: LSM6DSO32TR, Package_LGA:LGA-14_3x2.5mm_P0.5mm_LayoutBorder3x4y, symbol Io_Symbols:LSM6DSO32
- added U5: RFM95W-915S2, symbol RF_Module:RFM95W-915S2
- C1, C2, C3, C4: footprint (none) -> Capacitor_SMD:C_0402_1005Metric
- C10, C14, C15, C16, C8: renamed from C?; footprint (none) -> Capacitor_SMD:C_0402_1005Metric
- C11, C13, C6, C7, C9: renamed from C?; footprint (none) -> Capacitor_SMD:C_0603_1608Metric
- C5: footprint (none) -> Capacitor_SMD:C_0603_1608Metric
- F1: value Fuse (3A) -> 0ABA-2000-TN
- IC1: footprint SOT95P280X90-6N -> Footprints:SOT95P280X90-6N
- gave numbers to parts that had none: 9
Connections:
- net SW- is gone; now on an unnamed net: IC1.2 (EN)
- net +3.3V: now also C12.1, C19.1, C20.1, C21.1, C22.1, C23.1, C24.1, C25.1, C26.1, D2.2 (A), FB1.2, J1.1 (Pin_1), J2.4 (VDD), J4.1 (Pin_1), R22.1, U4.12 (CS)
- net GND: now also C12.2, C17.2, C18.2, C19.2, C20.2, C21.2, C22.2, C23.2, C26.2, IC2.10 (VDD), IC2.3 (VSS_1), IC2.8 (VSS_2), IC2.9 (VSS_3), J1.4 (Pin_4), J2.6 (VSS), J4.4 (Pin_4), J5.2 (Pin_2), J8.2 (Ext), Q2.1 (S), Q2.2 (S), Q2.3 (S), Q3.1 (S), Q3.2 (S), Q3.3 (S), Q4.1 (S), Q4.2 (S), Q4.3 (S), Q5.1 (S), Q5.2 (S), Q5.3 (S), R11.2, R13.2, R15.2, R17.2, R20.2, R6.2, R7.2, R8.2, R9.2, U3.1 (GND), U3.10 (GND), U3.11 (GND), U3.15 (GND), U3.16 (GND), U3.17 (VCC), U3.2 (VCC_IO), U3.20 (GND), U3.4 (GND), U3.5 (GND), U3.6 (GND), U4.1 (SDO/SA0), U4.2 (SDX), U4.3 (SCX), U4.5 (VDDIO), U4.6 (GND), U4.7 (GND), U4.8 (VDD), U5.1 (GND), U5.10 (GND), U5.8 (GND); no longer U1.13 (VDDA)
- net I2C1_SCL: now also U4.13 (SCL)
- net I2C1_SDA: now also U4.14 (SDA)
- net I2C2_SCL: now also IC2.2 (SCK), U3.12 (SCL)
- net I2C2_SDA: now also U3.9 (SDA)
- net I2C3_SCL: now also J1.3 (Pin_3)
- net I2C3_SDA: now also J1.2 (Pin_2)
- net PYRO1: now also R2.1
- net PYRO1_DET: now also R10.2, R11.1
- net PYRO2: now also R3.1
- net PYRO2_DET: now also R12.2, R13.1
- net PYRO3: now also R4.1
- net PYRO3_DET: now also R14.2, R15.1
- net PYRO4: now also R5.1
- net PYRO4_DET: now also R16.2, R17.1
- net SDMMC_CMD: now also J2.3 (CMD)
- net SDMMC_D0: now also J2.7 (DAT0)
- net SDMMC_D1: now also J2.8 (DAT1)
- net SDMMC_D2: now also J2.1 (DAT2)
- net SDMMC_D3: now also J2.2 (DAT3/CD)
- net SDMMC_DET: now also J2.9 (DET_B)
- net SPI1_MISO: now also U5.2 (MISO)
- net SPI1_MOSI: now also U5.3 (MOSI)
- net SPI1_NSS: now also U5.5 (NSS)
- net SPI1_SCK: now also U5.4 (SCK)
- net SPI2_MISO: now also U1.35 (PB14), IC2.5 (SDO); no longer U1.10 (PC2)
- net SPI2_MOSI: now also U1.36 (PB15), IC2.4 (SDI); no longer U1.11 (PC3)
- net SPI2_NSS: now also IC2.6 (CSB)
- net SWCLK: now also J4.3 (Pin_3)
- net SWDIO: now also J4.2 (Pin_2)
- net USB_D+: now also R22.2
- net BATT+ renamed ARM
- net ARM: now also J3.2 (Pin_2), J3.4 (Pin_4), J3.6 (Pin_6), J3.8 (Pin_8), J6.2 (Pin_2)
- net BATT_DET: no longer names the net of U1.24 (PC4)
- net SDMMC_CK renamed SDMMC_CLK
- net SDMMC_CLK: now also J2.5 (CLK)
- new net: Q3.4 (G), R3.2, R7.1
- new net: J8.1 (In), U5.9 (ANT)
- new net: Q2.4 (G), R2.2, R6.1
- new net: C24.2, IC2.1 (VDDIO)
- new net: Q5.4 (G), R5.2, R9.1
- new net: D2.1 (K), R20.1
- new net: C25.2, U5.13 (3.3V)
- new net: Q4.4 (G), R4.2, R8.1
- new net +3.3VA: C17.1, C18.1, FB1.1, U1.13 (VDDA)
- new net BATT: J5.1 (Pin_1), J6.1 (Pin_1)
- new net PYRO1_SW: J3.1 (Pin_1), Q2.5 (D), R10.1
- new net PYRO2_SW: J3.3 (Pin_3), Q3.5 (D), R12.1
- new net PYRO3_SW: J3.5 (Pin_5), Q4.5 (D), R14.1
- new net PYRO4_SW: J3.7 (Pin_7), Q5.5 (D), R16.1
- new net RF_RESET: U5.6 (RESET)
- no-connect marks 2 -> 33
Other:
- note added: "3V3 Linear Regulator"
- note added: "40MHz Crystal"
- note added: "5V Buck Converter"
- note added: "ADC Power Filtering"
- note added: "ALTIMETER"
- note added: "Arming"
- note added: "Battery"
- note added: "Device expects 2S LiPo Battery (6.4-8.4V, 7.4V Nominal)"
- note added: "External I2C"
- note added: "Filtering Capactors"
- note added: "GPS"
- note added: "IMU/TEMP"
- note added: "MCU"
- note added: "Micro USB Connector"
- note added: "MicroSD Card"
- note added: "PERIPHERALS"
- note added: "POWER"
- note added: "PYROS"
- note added: "Peripheral Assignments: I2C1: IMU I2C2: GPS I2C3: External Interface SPI1: RF SPI2: Altimeter"
- note added: "Pyro 1"
- note added: "Pyro 2"
- note added: "Pyro 3"
- note added: "Pyro 4"
- note added: "Pyro Connections"
- note added: "RF"
- note added: "SWD"
- moved on the sheet: C1, C10, C11, C13, C14, C15, C16, C2, C3, C4, C5, C6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

Commit message: Schematic adjustments
Parts:
- removed F1: 0ABA-2000-TN, symbol Device:Fuse
- removed R2, R3, R4, R5: 1K, symbol Device:R
- added U?: USBLC6-2SC6, Package_TO_SOT_SMD:SOT-23-6, symbol Power_Protection:USBLC6-2SC6
- C1, C12, C15, C2, C20, C21, C22, C23, C24, C25, C26, C3, C4, C8: value 100nf -> 100n
- C10: value 47pf -> 47p
- C11, C13: value 22uf -> 22u
- C14, C16: value 10pf -> 10p
- C5, C6, C7, C9: value 10uf -> 10u
- R1, R6, R7, R8, R9: value 100K -> 30.1K
- R20, R22: value 1.5k -> 1.5K
Connections:
- net ARM: now also C6.1, IC1.2 (EN), IC1.3 (VIN)
- net GND: now also U?.2 (GND)
- net I2C2_SCL: no longer IC2.2 (SCK)
- net PYRO1: now also Q2.4 (G), R6.1
- net PYRO2: now also Q3.4 (G), R7.1
- net PYRO3: now also Q4.4 (G), R8.1
- net PYRO4: now also Q5.4 (G), R9.1
- net SPI2_SCK: now also IC2.2 (SCK)
- net USB_D+: now also U?.1 (I/O1); no longer R22.2, U1.45 (PA12)
- net USB_D-: now also U?.3 (I/O2); no longer U1.44 (PA11)
- net VBUS: now also U?.5 (VBUS)
- net at C10.1, IC1.1 (FB): no longer R18.2, R19.1
- net +3.3VA: no longer names the net of C17.1, C18.1, FB1.1, U1.13 (VDDA)
- new net: R18.2, R19.1
- new net USB_ESD_D+: R22.2, U1.45 (PA12), U?.6 (I/O1)
- new net USB_ESD_D-: U1.44 (PA11), U?.4 (I/O2)
- no-connect marks 33 -> 35
Other:
- note added: "Micro USB and ESD"
- note added: "Note: ADC "zero" voltage is 2.0V Voltage dividers are tuned to provide 2.0V-2.6V with BATT at 6.4-8.4V"
- note added: "Note: Device expects 2S LiPo Battery (6.4-8.4V, 7.4V Nominal)"
- note removed: "Device expects 2S LiPo Battery (6.4-8.4V, 7.4V Nominal)"
- note removed: "Micro USB Connector"
- moved on the sheet: C1, C10, C11, C12, C13, C14, C15, C16, C17, C18, C19, C2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

Commit message: Started PCB design
Parts:
- D2: footprint (none) -> LED_SMD:LED_0603_1608Metric
- FB1: footprint (none) -> Inductor_SMD:L_0201_0603Metric
- IC1: footprint Footprints:SOT95P280X90-6N -> Package_TO_SOT_SMD:TSOT-23-6
- IC2: footprint BMP390 -> Io_Footprints:BMP390
- J1: footprint (none) -> Connector_PinHeader_2.54mm:PinHeader_1x04_P2.54mm_Vertical
- J2: renamed from J3; footprint (none) -> TerminalBlock_TE-Connectivity:TerminalBlock_TE_282834-8_1x08_P2.54mm_Horizontal
- J3: renamed from J4; footprint (none) -> Connector_PinHeader_2.54mm:PinHeader_1x04_P2.54mm_Vertical
- J4: renamed from J5; footprint (none) -> TerminalBlock_TE-Connectivity:TerminalBlock_TE_282834-2_1x02_P2.54mm_Horizontal
- J5: renamed from J6; footprint (none) -> TerminalBlock_TE-Connectivity:TerminalBlock_TE_282834-2_1x02_P2.54mm_Horizontal
- J6: renamed from J2; footprint (none) -> Io_Footprints:MEM2075-00-140-01-A
- J7: footprint (none) -> Io_Footprints:KMMXBSMT35SB30TR
- J8: value EMPCB.SMAFSTJ.B.HT -> 0732511151; footprint (none) -> Connector_Coaxial:SMA_Molex_73251-1153_EdgeMount_Horizontal
- L1: footprint (none) -> Inductor_SMD:L_0805_2012Metric
- R1: value 30.1K -> 30.1k; footprint (none) -> Resistor_SMD:R_0402_1005Metric
- R10: renamed from R14; footprint (none) -> Resistor_SMD:R_0402_1005Metric
- R11: renamed from R15; footprint (none) -> Resistor_SMD:R_0603_1608Metric
- R12: renamed from R16; footprint (none) -> Resistor_SMD:R_0402_1005Metric
- R13: renamed from R17; footprint (none) -> Resistor_SMD:R_0603_1608Metric
- R14: renamed from R18; value 30.1K -> 30.1k; footprint (none) -> Resistor_SMD:R_0402_1005Metric
- R15: renamed from R19; value 158K -> 158k; footprint (none) -> Resistor_SMD:R_0805_2012Metric
- R16: renamed from R20; value 1.5K -> 1.5k; footprint (none) -> Resistor_SMD:R_0402_1005Metric
- R17: renamed from R21; value 10K -> 10k; footprint (none) -> Resistor_SMD:R_0402_1005Metric
- R18: renamed from R22; value 1.5K -> 1.5k; footprint (none) -> Resistor_SMD:R_0402_1005Metric
- R2: renamed from R6; value 30.1K -> 30.1k; footprint (none) -> Resistor_SMD:R_0402_1005Metric
- R3: renamed from R7; value 30.1K -> 30.1k; footprint (none) -> Resistor_SMD:R_0402_1005Metric
- R4: renamed from R8; value 30.1K -> 30.1k; footprint (none) -> Resistor_SMD:R_0402_1005Metric
- R5: renamed from R9; value 30.1K -> 30.1k; footprint (none) -> Resistor_SMD:R_0402_1005Metric
- R6: renamed from R10; footprint (none) -> Resistor_SMD:R_0402_1005Metric
- R7: renamed from R11; footprint (none) -> Resistor_SMD:R_0603_1608Metric
- R8: renamed from R12; footprint (none) -> Resistor_SMD:R_0402_1005Metric
- R9: renamed from R13; footprint (none) -> Resistor_SMD:R_0603_1608Metric
- SW1: value SW_SPDT -> LSSM12-40-P-V-T/R; footprint (none) -> Io_Footprints:LSSM1240PVTR
- U5: footprint (none) -> Io_Footprints:RFM95W-915S2
- Y1: footprint (none) -> Crystal:Crystal_SMD_2016-4Pin_2.0x1.6mm
- gave numbers to parts that had none: 1
- renumbered C6 to C1, C3 to C10, C15 to C11, C16 to C12, C2 to C13, C1 to C14, C4 to C15, C17 to C16, C18 to C17, C19 to C18, C12 to C19, C7 to C2, C21 to C20, C23 to C21, C25 to C22, C24 to C23, C26 to C24, C22 to C25, C20 to C26, C8 to C3, C9 to C4, C10 to C5, C11 to C6, C13 to C7, C5 to C8, C14 to C9, U2 to U1, U1 to U2, U3 to U6
Connections:
- net +3.3V: now also IC2.1 (VDDIO), IC2.10 (VDD), U2.1 (VBAT), U2.19 (VDD), U2.32 (VDD), U2.48 (VDDUSB), U2.64 (VDD), U4.5 (VDDIO), U4.8 (VDD), U5.13 (3.3V), U6.17 (VCC), U6.2 (VCC_IO), U6.3 (V_BCKP)
- net ARM: now also J5.1 (Pin_1); no longer J5.2 (Pin_2)
- net BATT: now also J5.2 (Pin_2); no longer J5.1 (Pin_1)
- net GND: now also C22.2, C23.2; no longer IC2.10 (VDD), U2.1 (VBAT), U2.19 (VDD), U2.32 (VDD), U2.48 (VDDUSB), U2.64 (VDD), U4.5 (VDDIO), U4.8 (VDD), U6.17 (VCC), U6.2 (VCC_IO)
- net RF_RESET: now also U2.24 (PC4)
- no-connect marks 35 -> 34
Other:
- moved on the sheet: C10, C13, C14, C15, C16, C17, C18, C20, C21, C22, C23, C24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

Commit message: Intermediate avionics update
Parts:
- L1: footprint Inductor_SMD:L_0805_2012Metric -> Inductor_SMD:L_Bourns_SRR1260
Other:
- note added: "No battery drain data has been collected. For each device, we will be plugging in the device to a fully-charged battery, attaching voltmeter leads to the battery connections or wires, and then measuring the time for the battery voltage to dip below acceptable levels (generally the battery's nominal voltage to prevent full discharge + battery damage). Low-resolution video data will be recorded for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"
Changed lines of the file:
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@@
     (effects (font (size 1.9 1.9) italic) (justify left bottom))
+  )
+  (text "No battery drain data has been collected. \n\nFor each device, we will be plugging in the device to a fully-charged battery, attaching voltmeter leads to the battery connections or wires, and then measuring the time for the battery voltage to dip below acceptable levels (generally the battery's nominal voltage to prevent full discharge + battery damage). Low-resolution video data will be recorded for the test to provide timestamps for expected battery voltages - this will allow us to provide battery life estimates on our SRAD flight computer.\n"
+    (at -33.02 0 0)
+    (effects (font (size 1.27 1.27)) (justify left bottom))
   )
   (text "PERIPHERALS" (at 111.76 171.45 0)
@@
     (property "Reference" "L1" (id 0) (at 76.2 41.91 90))
     (property "Value" "6.8uH" (id 1) (at 76.2 44.45 90))
-    (property "Footprint" "Inductor_SMD:L_0805_2012Metric" (id 2) (at 76.2 46.99 0)
+    (property "Footprint" "Inductor_SMD:L_Bourns_SRR1260" (id 2) (at 76.2 46.99 0)
       (effects (font (size 1.27 1.27)) hide)
     )
@@
     )
     (path "/3d8c9830-3767-492e-962f-52b62edeef1e"
-      (reference "L1") (unit 1) (value "6.8uH") (footprint "Inductor_SMD:L_0805_2012Metric")
+      (reference "L1") (unit 1) (value "6.8uH") (footprint "Inductor_SMD:L_Bourns_SRR1260")
     )
     (path "/5d393dfc-be03-4118-b95f-9038fa31eed2"

Commit message: Redesigned with 4-layer board
Parts:
- removed Q2, Q3, Q4, Q5: CSD17578Q5A, Package_TO_SOT_SMD:TDSON-8-1, symbol Transistor_FET:CSD17578Q5A
- added Q2, Q3, Q4, Q5: DMG2302U, Package_TO_SOT_SMD:SOT-23, symbol Transistor_FET:DMG2302U
Connections:
- net GND: now also Q2.2 (S), Q3.2 (S), Q4.2 (S), Q5.2 (S)
- net PYRO1: now also Q2.1 (G)
- net PYRO1_SW: now also Q2.3 (D)
- net PYRO2: now also Q3.1 (G)
- net PYRO2_SW: now also Q3.3 (D)
- net PYRO3: now also Q4.1 (G)
- net PYRO3_SW: now also Q4.3 (D)
- net PYRO4: now also Q5.1 (G)
- net PYRO4_SW: now also Q5.3 (D)
- net USB_D+: now also U3.3 (I/O2); no longer U3.1 (I/O1)
- net USB_D-: now also U3.1 (I/O1); no longer U3.3 (I/O2)
- net USB_ESD_D+: now also U3.4 (I/O2); no longer U3.6 (I/O1)
- net USB_ESD_D-: now also U3.6 (I/O1); no longer U3.4 (I/O2)
- net VDDA: now reaches C16.1, C17.1, FB1.1, U2.13 (VDDA)
- net RF_ANT: now reaches J8.1 (In), U5.9 (ANT)
- net 5V_I: now reaches C3.1, IC1.5 (SW), L1.1
- net 5V_C: now reaches C3.2, IC1.6 (BST)
- net 5V_R: now reaches R14.2, R15.1
- net LDO_LED: now reaches D2.1 (K), R16.1
- net LDO_D: now reaches C2.1, D1.1 (K), U1.1 (VI)
- net RF_DIO0: now reaches U5.14 (DIO0)
- net RF_DIO0: now also U2.41 (PA8)
- net RF_DIO1: now reaches U5.15 (DIO1)
- net RF_DIO1: now also U2.42 (PA9)
- net RF_DIO5: now reaches U5.7 (DIO5)
- net RF_DIO5: now also U2.43 (PA10)
- no-connect marks 34 -> 28
Other:
- note removed: "No battery drain data has been collected. For each device, we will be plugging in the device to a fully-charged battery, attaching voltmeter leads to the battery connections or wires, and then measuring the time for the battery voltage to dip below acceptable levels (generally the battery's nominal voltage to prevent full discharge + battery damage). Low-resolution video data will be recorded for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"
- moved on the sheet: J8
